Commit message: fixed assembly

File: src/my_robot_description/urdf/my_robot.urdf.xacro (robot description, xacro)
@@ -25,5 +25,5 @@
         <mesh filename="file:///home/parsa/ros2_urdf_ws/src/my_robot_description/meshes//torso_joint_f.dae" scale="0.01 0.01 0.01"/>
       </geometry>
-      <origin xyz="-0.935 -0.93 -0.895" rpy="0 0 0"/>
+      <origin xyz="-0.93 -0.93 -0.91" rpy="0 0 0"/>
     </visual>
     <collision>
@@ -31,5 +31,5 @@
         <mesh filename="file:///home/parsa/ros2_urdf_ws/src/my_robot_description/meshes//torso_joint_f.dae" scale="0.01 0.01 0.01"/>
       </geometry>
-      <origin xyz="-0.935 -0.93 -0.895" rpy="0 0 0"/>
+      <origin xyz="-0.93 -0.93 -0.91" rpy="0 0 0"/>
     </collision>
     <inertial>
@@ -51,5 +51,5 @@
         <mesh filename="file:///home/parsa/ros2_urdf_ws/src/my_robot_description/meshes//torso_joint_f.dae" scale="0.01 0.01 0.01"/>
       </geometry>
-      <origin xyz="-0.935 -0.93 -0.895" rpy="0 0 0"/>
+      <origin xyz="-0.935 -0.93 -0.91" rpy="0 0 0"/>
     </visual>
     <collision>
@@ -57,5 +57,5 @@
         <mesh filename="file:///home/parsa/ros2_urdf_ws/src/my_robot_description/meshes//torso_joint_f.dae" scale="0.01 0.01 0.01"/>
       </geometry>
-      <origin xyz="-0.935 -0.93 -0.895" rpy="0 0 0"/>
+      <origin xyz="-0.935 -0.93 -0.91" rpy="0 0 0"/>
     </collision>
     <inertial>
@@ -68,5 +68,5 @@
     <parent link="base_link" />
     <child link="torso_joint_f_2" />
-    <origin xyz="-0.428 -0.658 0.894" rpy="0.0 0.0 -3.14"/>
+    <origin xyz="-0.435 -0.658 0.894" rpy="0.0 0.0 -3.14"/>
     <axis xyz="0 0 1"/>
     <limit lower="-1.57" upper="1.57" velocity="100" effort="100"/>
@@ -77,5 +77,5 @@
         <mesh filename="file:///home/parsa/ros2_urdf_ws/src/my_robot_description/meshes//torso_joint_b.dae" scale="0.01 0.01 0.01"/>
       </geometry>
-      <origin xyz="-1.43 -0.93 -0.895" rpy="0 0 0"/>
+      <origin xyz="-1.45 -0.93 -0.91" rpy="0 0 0"/>
     </visual>
     <collision>
@@ -83,5 +83,5 @@
         <mesh filename="file:///home/parsa/ros2_urdf_ws/src/my_robot_description/meshes//torso_joint_b.dae" scale="0.01 0.01 0.01"/>
       </geometry>
-      <origin xyz="-1.43 -0.93 -0.895" rpy="0 0 0"/>
+      <origin xyz="-1.45 -0.93 -0.91" rpy="0 0 0"/>
     </collision>
     <inertial>
@@ -103,5 +103,5 @@
         <mesh filename="file:///home/parsa/ros2_urdf_ws/src/my_robot_description/meshes//torso_joint_b.dae" scale="0.01 0.01 0.01"/>
       </geometry>
-      <origin xyz="-1.43 -0.93 -0.895" rpy="0 0 0"/>
+      <origin xyz="-1.45 -0.93 -0.91" rpy="0 0 0"/>
     </visual>
       <collision>
@@ -109,5 +109,5 @@
         <mesh filename="file:///home/parsa/ros2_urdf_ws/src/my_robot_description/meshes//torso_joint_b.dae" scale="0.01 0.01 0.01"/>
       </geometry>
-      <origin xyz="-1.43 -0.93 -0.895" rpy="0 0 0"/>
+      <origin xyz="-1.45 -0.93 -0.91" rpy="0 0 0"/>
     </collision>
     <inertial>
@@ -129,11 +129,11 @@
         <mesh filename="file:///home/parsa/ros2_urdf_ws/src/my_robot_description/meshes//femur.dae" scale="0.01 0.01 0.01"/>
       </geometry>
-      <origin xyz="-0.77 -1.14 -0.8" rpy="0 0 0"/>
-    </visual>
-    <collision>
-      <geometry>
-        <mesh filename="file:///home/parsa/ros2_urdf_ws/src/my_robot_description/meshes//femur.dae" scale="0.01 0.01 0.01"/>
-      </geometry>
-      <origin xyz="-0.77 -1.14 -0.8" rpy="0 0 0"/>
+      <origin xyz="-0.74 -1.16 -0.81" rpy="0 0 0"/>
+    </visual>
+    <collision>
+      <geometry>
+        <mesh filename="file:///home/parsa/ros2_urdf_ws/src/my_robot_description/meshes//femur.dae" scale="0.01 0.01 0.01"/>
+      </geometry>
+      <origin xyz="-0.74 -1.16 -0.81" rpy="0 0 0"/>
       </collision>
       <inertial>
@@ -146,5 +146,5 @@
     <parent link="torso_joint_f_1" />
     <child link="femur_1" />
-    <origin xyz="-0.197 0.229 -0.043" rpy="0.0 0.0 0.0"/>
+    <origin xyz="-0.191 0.229 -0.099" rpy="0.0 0.0 0.0"/>
     <axis xyz="1 0 0"/>
     <limit lower="-1.57" upper="1.57" velocity="100" effort="100"/>
@@ -155,11 +155,11 @@
         <mesh filename="file:///home/parsa/ros2_urdf_ws/src/my_robot_description/meshes//femur.dae" scale="0.01 0.01 0.01"/>
       </geometry>
-      <origin xyz="-0.73 -1.17 -0.8" rpy="0 0 0"/>
-    </visual>
-    <collision>
-      <geometry>
-        <mesh filename="file:///home/parsa/ros2_urdf_ws/src/my_robot_description/meshes//femur.dae" scale="0.01 0.01 0.01"/>
-      </geometry>
-      <origin xyz="-0.73 -1.17 -0.8" rpy="0 0 0"/>
+      <origin xyz="-0.74 -1.17 -0.81" rpy="0 0 0"/>
+    </visual>
+    <collision>
+      <geometry>
+        <mesh filename="file:///home/parsa/ros2_urdf_ws/src/my_robot_description/meshes//femur.dae" scale="0.01 0.01 0.01"/>
+      </geometry>
+      <origin xyz="-0.74 -1.17 -0.81" rpy="0 0 0"/>
     </collision>
       <inertial>
@@ -172,5 +172,5 @@
     <parent link="torso_joint_f_2" />
     <child link="femur_2" />
-    <origin xyz="-0.187 0.231 -0.042" rpy="0.0 0.0 0.0"/>
+    <origin xyz="-0.191 0.231 -0.099" rpy="0.0 0.0 0.0"/>
     <axis xyz="1 0 0"/>
     <limit lower="-1.57" upper="1.57" velocity="100" effort="100"/>
@@ -181,11 +181,11 @@
         <mesh filename="file:///home/parsa/ros2_urdf_ws/src/my_robot_description/meshes//femur.dae" scale="0.01 0.01 0.01"/>
       </geometry>
-      <origin xyz="-0.774 -1.17 -0.81" rpy="0 0 0"/>
-    </visual>
-    <collision>
-      <geometry>
-        <mesh filename="file:///home/parsa/ros2_urdf_ws/src/my_robot_description/meshes//femur.dae" scale="0.01 0.01 0.01"/>
-      </geometry>
-      <origin xyz="-0.774 -1.17 -0.81" rpy="0 0 0"/>
+      <origin xyz="-0.76 -1.17 -0.77" rpy="0 0 0"/>
+    </visual>
+    <collision>
+      <geometry>
+        <mesh filename="file:///home/parsa/ros2_urdf_ws/src/my_robot_description/meshes//femur.dae" scale="0.01 0.01 0.01"/>
+      </geometry>
+      <origin xyz="-0.76 -1.17 -0.77" rpy="0 0 0"/>
     </collision>
       <inertial>
@@ -207,11 +207,11 @@
         <mesh filename="file:///home/parsa/ros2_urdf_ws/src/my_robot_description/meshes//femur.dae" scale="0.01 0.01 0.01"/>
       </geometry>
-      <origin xyz="-0.774 -1.17 -0.81" rpy="0 0 0"/>
-    </visual>
-    <collision>
-      <geometry>
-        <mesh filename="file:///home/parsa/ros2_urdf_ws/src/my_robot_description/meshes//femur.dae" scale="0.01 0.01 0.01"/>
-      </geometry>
-      <origin xyz="-0.774 -1.17 -0.81" rpy="0 0 0"/>
+      <origin xyz="-0.76 -1.17 -0.77" rpy="0 0 0"/>
+    </visual>
+    <collision>
+      <geometry>
+        <mesh filename="file:///home/parsa/ros2_urdf_ws/src/my_robot_description/meshes//femur.dae" scale="0.01 0.01 0.01"/>
+      </geometry>
+      <origin xyz="-0.76 -1.17 -0.77" rpy="0 0 0"/>
     </collision>
       <inertial>
@@ -233,5 +233,5 @@
         <mesh filename="file:///home/parsa/ros2_urdf_ws/src/my_robot_description/meshes//foot-f-1.dae" scale="0.01 0.01 0.01"/>
       </geometry>
-      <origin xyz="0.68 1.47 -0.75" rpy="0 0 3.14"/>
+      <origin xyz="0.741 1.54 -0.8" rpy="0 0 3.14"/>
     </visual>
     <collision>
@@ -239,5 +239,5 @@
         <mesh filename="file:///home/parsa/ros2_urdf_ws/src/my_robot_description/meshes//foot-f-1.dae" scale="0.01 0.01 0.01"/>
       </geometry>
-      <origin xyz="0.68 1.47 -0.75" rpy="0 0 3.14"/>
+      <origin xyz="0.741 1.54 -0.8" rpy="0 0 3.14"/>
     </collision>
     <inertial>
@@ -250,5 +250,5 @@
   <parent link="femur_1" />
   <child link="foot-f-1" />
-    <origin xyz="-0.04 0.4 -0.02" rpy="0 0 3.14"/>
+    <origin xyz="-0.013 0.368 -0.02" rpy="0 0 3.14"/>
     <axis xyz="1 0 0"/>
     <limit lower="-1.57" upper="1.57" velocity="100" effort="100"/>
@@ -259,5 +259,5 @@
         <mesh filename="file:///home/parsa/ros2_urdf_ws/src/my_robot_description/meshes//foot-f-1.dae" scale="0.01 0.01 0.01"/>
       </geometry>
-      <origin xyz="0.68 1.47 -0.75" rpy="0 0 3.14"/>
+      <origin xyz="0.741 1.54 -0.8" rpy="0 0 3.14"/>
     </visual>
     <collision>
@@ -265,5 +265,5 @@
         <mesh filename="file:///home/parsa/ros2_urdf_ws/src/my_robot_description/meshes//foot-f-1.dae" scale="0.01 0.01 0.01"/>
       </geometry>
-      <origin xyz="0.68 1.47 -0.75" rpy="0 0 3.14"/>
+      <origin xyz="0.741 1.54 -0.8" rpy="0 0 3.14"/>
     </collision>
     <inertial>
@@ -276,5 +276,5 @@
   <parent link="femur_2" />
   <child link="foot-f-2" />
-    <origin xyz="-0.023 0.38 -0.026" rpy="0 0 3.14"/>
+    <origin xyz="-0.013 0.368 -0.02" rpy="0 0 3.14"/>
     <axis xyz="1 0 0"/>
     <limit lower="-1.57" upper="1.57" velocity="100" effort="100"/>
@@ -285,5 +285,5 @@
         <mesh filename="file:///home/parsa/ros2_urdf_ws/src/my_robot_description/meshes//foot-b-1.dae" scale="0.01 0.01 0.01"/>
       </geometry>
-      <origin xyz="1.45 -1.37 0.84" rpy="-3.14 0 3.14"/>
+      <origin xyz="1.64 -1.54 0.84" rpy="-3.14 0 3.14"/>
     </visual>
     <collision>
@@ -291,5 +291,5 @@
         <mesh filename="file:///home/parsa/ros2_urdf_ws/src/my_robot_description/meshes//foot-b-1.dae" scale="0.01 0.01 0.01"/>
       </geometry>
-      <origin xyz="1.45 -1.37 0.84" rpy="-3.14 0 3.14"/>
+      <origin xyz="1.64 -1.54 0.84" rpy="-3.14 0 3.14"/>
     </collision>
     <inertial>
@@ -302,5 +302,5 @@
   <parent link="femur_3" />
   <child link="foot-b-1" />
-    <origin xyz="-0.023 0.38 -0.026" rpy="0 0 0"/>
+    <origin xyz="-0.013 0.368 -0.02" rpy="0 0 0"/>
     <axis xyz="1 0 0"/>
     <limit lower="-1.57" upper="1.57" velocity="100" effort="100"/>
@@ -311,5 +311,5 @@
         <mesh filename="file:///home/parsa/ros2_urdf_ws/src/my_robot_description/meshes//foot-b-1.dae" scale="0.01 0.01 0.01"/>
       </geometry>
-      <origin xyz="1.45 -1.37 0.84" rpy="-3.14 0 3.14"/>
+      <origin xyz="1.64 -1.54 0.84" rpy="-3.14 0 3.14"/>
     </visual>
     <collision>
@@ -317,5 +317,5 @@
         <mesh filename="file:///home/parsa/ros2_urdf_ws/src/my_robot_description/meshes//foot-b-1.dae" scale="0.01 0.01 0.01"/>
       </geometry>
-      <origin xyz="1.45 -1.37 0.84" rpy="-3.14 0 3.14"/>
+      <origin xyz="1.64 -1.54 0.84" rpy="-3.14 0 3.14"/>
     </collision>
     <inertial>
@@ -328,5 +328,5 @@
   <parent link="femur_4" />
   <child link="foot-b-2" />
-    <origin xyz="-0.023 0.38 -0.026" rpy="0 0 0"/>
+    <origin xyz="-0.013 0.368 -0.02" rpy="0 0 0"/>
     <axis xyz="1 0 0"/>
     <limit lower="-1.57" upper="1.57" velocity="100" effort="100"/>
